File: SensorNodeCircuit-V2/SensorNodeCircuit.kicad_pcb (KiCad board)
At the start: 2 copper layers, 68.4 x 34.9 mm, 26 parts, among them J1 USB_B_Micro, J2 FTDI, J3 ExtraPins, J4 ProgJump, J5 PWR, J6 MuxExtra, SW1 ResetButton, U1 AMS1117-3.3, U2 ESP-12F, U3 CD4051B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

Commit message: Tidied up pcb
Parts:
- added REF**: MountingHole_2.2mm_M2_ISO14580_Pad, MountingHole:MountingHole_2.2mm_M2_ISO14580_Pad, F.Cu at (105.0, 79.5)
- added REF**: MountingHole_2.7mm_Pad, MountingHole:MountingHole_2.7mm_Pad, F.Cu at (105.5, 107.0)
- added REF**: MountingHole_2.7mm_Pad, MountingHole:MountingHole_2.7mm_Pad, F.Cu at (166.0, 107.1)
- U4: value LM35-LP -> LM35
Routing:
- net GND: track 11.6 -> 13.7 mm, vias 54 -> 14
Other:
- board text added: "+3.3"
- board text added: "0"
- board text added: "1"
- board text removed: "+"
- board text removed: "-"
- board text removed: "SCLK"

Commit message: Added sensornode pcb 3d render
Parts:
- removed the REF** at (105.0, 79.5)
- removed the REF** at (105.5, 107.0)
- removed the REF** at (166.0, 107.1)
- added REF**: MountingHole_2.5mm_Pad, MountingHole:MountingHole_2.5mm_Pad, F.Cu at (105.5, 107.0)
- added REF**: MountingHole_2.5mm_Pad, MountingHole:MountingHole_2.5mm_Pad, F.Cu at (166.0, 107.0)
Other:
- board text added: "CLK"
Changed lines of the file:
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@@
   (general
     (thickness 1.6)
-    (drawings 30)
+    (drawings 31)
     (tracks 226)
     (zones 0)
-    (modules 29)
+    (modules 28)
     (nets 33)
   )
@@
     (mod_text_size 1 1)
     (mod_text_width 0.15)
-    (pad_size 1.6 0.6)
-    (pad_drill 0)
+    (pad_size 5 5)
+    (pad_drill 2.5)
     (pad_to_mask_clearance 0.051)
     (solder_mask_min_width 0.25)
@@
     (add_net TempOut)
   )
-  (module MountingHole:MountingHole_2.2mm_M2_ISO14580_Pad (layer F.Cu)
-    (at 105 79.5)
-    (descr "Mounting Hole 2.2mm, M2, ISO14580")
-    (tags "mounting hole 2.2mm m2 iso14580")
+  (module MountingHole:MountingHole_2.5mm_Pad (layer F.Cu)
+    (at 105.5 107)
+    (descr "Mounting Hole 2.5mm")
+    (tags "mounting hole 2.5mm")
     (attr virtual)
-    (fp_text reference REF** (at 0 -2.9) (layer F.SilkS) hide
-      (effects (font (size 1 1) (thickness 0.15)))
-    )
-    (fp_text value MountingHole_2.2mm_M2_ISO14580_Pad (at 0 2.9) (layer F.Fab)
-      (effects (font (size 1 1) (thickness 0.15)))
-    )
-    (fp_circle (center 0 0) (end 2.15 0) (layer F.CrtYd) (width 0.05))
-    (fp_circle (center 0 0) (end 1.9 0) (layer Cmts.User) (width 0.15))
+    (fp_text reference REF** (at 0 -3.5) (layer F.SilkS) hide
+      (effects (font (size 1 1) (thickness 0.15)))
+    )
+    (fp_text value MountingHole_2.5mm_Pad (at 0 3.5) (layer F.Fab)
+      (effects (font (size 1 1) (thickness 0.15)))
+    )
+    (fp_circle (center 0 0) (end 2.75 0) (layer F.CrtYd) (width 0.05))
+    (fp_circle (center 0 0) (end 2.5 0) (layer Cmts.User) (width 0.15))
     (fp_text user %R (at 0.3 0) (layer F.Fab)
       (effects (font (size 1 1) (thickness 0.15)))
     )
-    (pad 1 thru_hole circle (at 0 0) (size 3.8 3.8) (drill 2.2) (layers *.Cu *.Mask))
-  )
-  (module MountingHole:MountingHole_2.7mm_Pad (layer F.Cu)
-    (at 105.5 107)
-    (descr "Mounting Hole 2.7mm")
-    (tags "mounting hole 2.7mm")
+    (pad 1 thru_hole circle (at 0 0) (size 5 5) (drill 2.5) (layers *.Cu *.Mask)
+      (net 1 GND))
+  )
+  (module MountingHole:MountingHole_2.5mm_Pad (layer F.Cu)
+    (at 166 107)
+    (descr "Mounting Hole 2.5mm")
+    (tags "mounting hole 2.5mm")
     (attr virtual)
-    (fp_text reference REF** (at 0 -3.7) (layer F.SilkS) hide
-      (effects (font (size 1 1) (thickness 0.15)))
-    )
-    (fp_text value MountingHole_2.7mm_Pad (at 0 3.7) (layer F.Fab)
-      (effects (font (size 1 1) (thickness 0.15)))
-    )
-    (fp_circle (center 0 0) (end 2.95 0) (layer F.CrtYd) (width 0.05))
-    (fp_circle (center 0 0) (end 2.7 0) (layer Cmts.User) (width 0.15))
+    (fp_text reference REF** (at 0 -3.5) (layer F.SilkS) hide
+      (effects (font (size 1 1) (thickness 0.15)))
+    )
+    (fp_text value MountingHole_2.5mm_Pad (at 0 3.5) (layer F.Fab)
+      (effects (font (size 1 1) (thickness 0.15)))
+    )
+    (fp_circle (center 0 0) (end 2.75 0) (layer F.CrtYd) (width 0.05))
+    (fp_circle (center 0 0) (end 2.5 0) (layer Cmts.User) (width 0.15))
     (fp_text user %R (at 0.3 0) (layer F.Fab)
       (effects (font (size 1 1) (thickness 0.15)))
     )
-    (pad 1 thru_hole circle (at 0 0) (size 5.4 5.4) (drill 2.7) (layers *.Cu *.Mask))
-  )
-  (module MountingHole:MountingHole_2.7mm_Pad (layer F.Cu)
-    (at 166 107.1)
-    (descr "Mounting Hole 2.7mm")
-    (tags "mounting hole 2.7mm")
-    (attr virtual)
-    (fp_text reference REF** (at 0 -3.7) (layer F.SilkS) hide
-      (effects (font (size 1 1) (thickness 0.15)))
-    )
-    (fp_text value MountingHole_2.7mm_Pad (at 0 3.7) (layer F.Fab)
-      (effects (font (size 1 1) (thickness 0.15)))
-    )
-    (fp_circle (center 0 0) (end 2.95 0) (layer F.CrtYd) (width 0.05))
-    (fp_circle (center 0 0) (end 2.7 0) (layer Cmts.User) (width 0.15))
-    (fp_text user %R (at 0.3 0) (layer F.Fab)
-      (effects (font (size 1 1) (thickness 0.15)))
-    )
-    (pad 1 thru_hole circle (at 0 0) (size 5.4 5.4) (drill 2.7) (layers *.Cu *.Mask))
+    (pad 1 thru_hole circle (at 0 0) (size 5 5) (drill 2.5) (layers *.Cu *.Mask)
+      (net 1 GND))
   )
   (module Capacitor_SMD:C_1206_3216Metric_Pad1.42x1.75mm_HandSolder (layer F.Cu)
@@
     )
   )
+  (dimension 4 (width 0.15) (layer Dwgs.User)
+    (gr_text "4.000 mm" (at 173.3 109.25 270) (layer Dwgs.User)
+      (effects (font (size 1 1) (thickness 0.15)))
+    )
+    (feature1 (pts (xy 166 111.25) (xy 172.586421 111.25)))
+    (feature2 (pts (xy 166 107.25) (xy 172.586421 107.25)))
+    (crossbar (pts (xy 172 107.25) (xy 172 111.25)))
+    (arrow1a (pts (xy 172 111.25) (xy 171.413579 110.123496)))
+    (arrow1b (pts (xy 172 111.25) (xy 172.586421 110.123496)))
+    (arrow2a (pts (xy 172 107.25) (xy 171.413579 108.376504)))
+    (arrow2b (pts (xy 172 107.25) (xy 172.586421 108.376504)))
+  )
+  (dimension 4 (width 0.15) (layer Dwgs.User)
+    (gr_text "4.000 mm" (at 168 113.55) (layer Dwgs.User)
+      (effects (font (size 1 1) (thickness 0.15)))
+    )
+    (feature1 (pts (xy 170 106.25) (xy 170 112.836421)))
+    (feature2 (pts (xy 166 106.25) (xy 166 112.836421)))
+    (crossbar (pts (xy 166 112.25) (xy 170 112.25)))
+    (arrow1a (pts (xy 170 112.25) (xy 168.873496 112.836421)))
+    (arrow1b (pts (xy 170 112.25) (xy 168.873496 111.663579)))
+    (arrow2a (pts (xy 166 112.25) (xy 167.126504 112.836421)))
+    (arrow2b (pts (xy 166 112.25) (xy 167.126504 111.663579)))
+  )
+  (gr_text CLK (at 158.75 109.25 90) (layer F.SilkS)
+    (effects (font (size 0.8 0.8) (thickness 0.15)))
+  )
   (gr_text +5V (at 104 83) (layer F.SilkS)
     (effects (font (size 1 1) (thickness 0.15)))
@@
     (arrow2b (pts (xy 105.5 112) (xy 104.373496 112.586421)))
   )
-  (dimension 4 (width 0.15) (layer Dwgs.User)
-    (gr_text "4.000 mm" (at 172.3 109 90) (layer Dwgs.User)
-      (effects (font (size 1 1) (thickness 0.15)))
-    )
-    (feature1 (pts (xy 166 107) (xy 171.586421 107)))
-    (feature2 (pts (xy 166 111) (xy 171.586421 111)))
-    (crossbar (pts (xy 171 111) (xy 171 107)))
-    (arrow1a (pts (xy 171 107) (xy 171.586421 108.126504)))
-    (arrow1b (pts (xy 171 107) (xy 170.413579 108.126504)))
-    (arrow2a (pts (xy 171 111) (xy 171.586421 109.873496)))
-    (arrow2b (pts (xy 171 111) (xy 170.413579 109.873496)))
-  )
-  (dimension 4 (width 0.15) (layer Dwgs.User)
-    (gr_text "4.000 mm" (at 168 113.3) (layer Dwgs.User)
-      (effects (font (size 1 1) (thickness 0.15)))
-    )
-    (feature1 (pts (xy 166 107) (xy 166 112.586421)))
-    (feature2 (pts (xy 170 107) (xy 170 112.586421)))
-    (crossbar (pts (xy 170 112) (xy 166 112)))
-    (arrow1a (pts (xy 166 112) (xy 167.126504 111.413579)))
-    (arrow1b (pts (xy 166 112) (xy 167.126504 112.586421)))
-    (arrow2a (pts (xy 170 112) (xy 168.873496 111.413579)))
-    (arrow2b (pts (xy 170 112) (xy 168.873496 112.586421)))
-  )
   (dimension 34.9 (width 0.15) (layer Dwgs.User)
